Commit message: Update camera.xacro

File: Universal_Robots_ROS2_Description/urdf/camera.xacro (robot description, xacro)
@@ -33,28 +33,4 @@
         </visual>
     </link>
-    <!-- <gazebo reference="camera_link">
-        <material> Gazebo/black </material>
-        <sensor name="camera" type="camera">
-            <pose> 0 0 0 0 0 0 </pose>
-            <visualize>true</visualize>
-            <update_rate>60</update_rate>
-            <always_on>1</always_on>
-            <camera>
-                <camera_info_topic>camera/camera_info</camera_info_topic>
-                <vertical_fov>1.3</vertical_fov>
-                <image>
-                    <format>R8G8B8</format>
-                    <width>1920</width>
-                    <height>1080</height>
-                </image>
-                <clip>
-                    <near>0.01</near>
-                    <far>10.0</far>
-                </clip>
-             </camera>
-             <topic>camera/image_raw</topic>
-             <gz_frame_id>camera_optical_link</gz_frame_id>
-        </sensor>
-    </gazebo> -->
     <gazebo reference="camera_link">
         <material> Gazebo/black </material>
@@ -88,6 +64,4 @@
             </depth_camera>
             <topic>camera</topic>
-            <!-- <depth_topic>camera/depth/image_raw</depth_topic>
-            <point_cloud_topic>camera/depth/points</point_cloud_topic> -->
             <gz_frame_id>camera_optical_link</gz_frame_id>
         </sensor>
@@ -152,10 +126,4 @@
             </geometry>
         </visual>
-        <!-- <collision>
-            <geometry>
-                Reference your .dae file for collision geometry as well
-                <mesh filename="package://ur_simulation_gz/models/ccs2_outlet/ccs1_plug.dae" scale="0.025 0.025 0.025"/>
-            </geometry>
-        </collision> -->
         <inertial>
             <mass value="0.1"/>

Commit message: Update camera.xacro

File: Universal_Robots_ROS2_Description/urdf/camera.xacro (robot description, xacro)
@@ -95,6 +95,6 @@
     <gazebo reference="flashlight_optical_link">
         <light type="spot" name="arm_light">
-            <pose>0 0 0 0 0 0</pose>  <!-- Relative to the link -->
-            <diffuse>0.5 0.5 0.5 1</diffuse>  <!-- grey light -->
+            <pose>0 0 0 0 0 0</pose>
+            <diffuse>0.5 0.5 0.5 1</diffuse>
             <specular>0.1 0.1 0.1 1</specular>
             <attenuation>
@@ -111,5 +111,5 @@
             </spot>
             <cast_shadows>true</cast_shadows>
-            <visualize>false</visualize> <!-- Remove the green helper lines -->
+            <visualize>false</visualize>
         </light>
     </gazebo>
@@ -123,5 +123,4 @@
             <geometry>
                 <mesh filename="package://ccs2_outlet/ccs1_plug.dae" scale="0.033 0.033 0.033"/>
-                <!-- <mesh filename="model://ccs2_outlet" scale="0.033 0.033 0.033"/> -->
             </geometry>
         </visual>
